File: kicad/m2ngff.kicad_pcb (KiCad board)
At the start: 2 copper layers, 85.1 x 74.1 mm, 10 parts

Commit message: update
Parts:
- added AE: NGFF_AE, ngff:NGFF_AE, F.Cu at (109.0, 94.6)
- added STOPs.top: NGFF-BM2230, m2ngff:m2-outer2230, F.Cu at (109.0, 94.6)
- moved REF** 110.1 mm to (241.1, 94.2)
- moved REF** 110.1 mm to (273.8, 94.7)
- moved STOPs.top 110.1 mm to (241.1, 94.2)
- moved STOPs.top 110.1 mm to (273.8, 94.7)
Other:
- board size 85.1 x 74.1 mm -> 186.7 x 26.7 mm

Commit message: update
Parts:
- added REF**: NGFF_AM, ngff:NGFF_AM, F.Cu at (275.3, 144.2)
- added REF**: NGFF_MEBA, ngff:NGFF_MEBA, F.Cu at (200.9, 194.0)
- added REF**: NGFF_ME, ngff:NGFF_ME, F.Cu at (239.0, 144.0)
- added STOPs.top: NGFF-BM2230, m2ngff:m2-outer2230, F.Cu at (239.0, 144.0)
- added STOPs.top: NGFF-BM2230, m2ngff:m2-outer2230, F.Cu at (200.9, 194.0)
- added STOPs.top: NGFF-BM2230, m2ngff:m2-outer2230, F.Cu at (275.3, 144.2)
- moved AE 82.7 mm to (173.8, 145.9)
- moved REF** 82.6 mm to (205.8, 145.3)
- moved STOPs.top 82.6 mm to (205.8, 145.3)
- moved STOPs.top 82.6 mm to (173.8, 145.9)
Other:
- board size 186.7 x 26.7 mm -> 123.6 x 125.8 mm
