File: kicad/E2250.kicad_pcb (KiCad board)
At the start: 2 copper layers, 22 x 46 mm, 2 parts

Commit message: update
Parts:
- removed E**: NGFF_E, NGFF:NGFF_E
- added REF**: STOP_A, ngff:NGFF_A, F.Cu at (115.0, 90.0)
Other:
- outline, holes or cut-outs redrawn
Changed lines of the file:
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@@
   )
   (net 0 "")
-  (footprint "NGFF:NGFF_2250" (layer "F.Cu")
+  (footprint "ngff:NGFF_A" (layer "F.Cu")
     (at 115 90)
     (attr through_hole)
-    (fp_text reference "STOPs.top" (at -8 -49) (layer "F.SilkS")
-      (effects (font (size 0.5 0.5) (thickness 0.125)))
-    )
-    (fp_text value "2250" (at -8 -47.5) (layer "F.SilkS")
+    (fp_text reference "REF**" (at 5.6 2.07) (layer "F.SilkS")
       (effects (font (size 1 1) (thickness 0.15)))
     )
-    (fp_line (start -11 -20) (end 11 -20) (layer "B.SilkS") (width 0.12))
-    (fp_line (start -11 -40) (end 11 -40) (layer "B.SilkS") (width 0.12))
-    (fp_line (start 0 0) (end 0 -30) (layer "Eco1.User") (width 0.01))
-    (fp_line (start 11 -50) (end 11 -4) (layer "Edge.Cuts") (width 0.05))
-    (fp_line (start 11 -50) (end -11 -50) (layer "Edge.Cuts") (width 0.05))
-    (fp_line (start -11 -50) (end -11 -4) (layer "Edge.Cuts") (width 0.05))
-    (fp_circle (center 0 -42) (end 1.5 -42) (layer "Edge.Cuts") (width 0.12) (fill none))
-    (fp_line (start -11 -50) (end -11 -4) (layer "F.CrtYd") (width 0.05))
-    (fp_line (start 11 -50) (end -11 -50) (layer "F.CrtYd") (width 0.05))
-    (fp_line (start 11 -50) (end 11 -4) (layer "F.CrtYd") (width 0.05))
-  )
-  (footprint "NGFF:NGFF_E" (layer "F.Cu")
-    (at 115 90)
-    (attr through_hole)
-    (fp_text reference "E**" (at 3.34 1.11) (layer "F.SilkS")
+    (fp_text value "STOP_A" (at -0.075 2.05) (layer "F.Fab")
       (effects (font (size 1 1) (thickness 0.15)))
     )
-    (fp_text value "NGFF_E" (at -3.04 1.18) (layer "F.Fab")
-      (effects (font (size 1 1) (thickness 0.15)))
-    )
-    (fp_text user "E" (at 2.61 -4.14) (layer "F.SilkS")
+    (fp_text user "A" (at 6.675 -4) (layer "B.SilkS")
       (effects (font (size 0.8 0.8) (thickness 0.15)))
     )
     (fp_poly (pts
-        (xy 3.225 0)
+        (xy 7.225 0)
         (xy 9.925 0)
         (xy 9.925 -2.5)
-        (xy 3.225 -2.5)
+        (xy 7.225 -2.5)
       ) (layer "B.Mask") (width 0.1) (fill solid))
     (fp_poly (pts
         (xy -9.925 0)
-        (xy 2.025 0)
-        (xy 2.025 -2.5)
+        (xy 6.025 0)
+        (xy 6.025 -2.5)
         (xy -9.925 -2.5)
       ) (layer "B.Mask") (width 0.1) (fill solid))
     (fp_poly (pts
+        (xy 7.225 0)
+        (xy 9.925 0)
+        (xy 9.925 -2)
+        (xy 7.225 -2)
+      ) (layer "F.Mask") (width 0.1) (fill solid))
+    (fp_poly (pts
         (xy -9.925 0)
-        (xy 2.025 0)
-        (xy 2.025 -2)
+        (xy 6.025 0)
+        (xy 6.025 -2)
         (xy -9.925 -2)
       ) (layer "F.Mask") (width 0.1) (fill solid))
-    (fp_poly (pts
-        (xy 3.225 0)
-        (xy 9.925 0)
-        (xy 9.925 -2)
-        (xy 3.225 -2)
-      ) (layer "F.Mask") (width 0.1) (fill solid))
+    (fp_line (start 7.225 0) (end 9.925 0) (layer "Edge.Cuts") (width 0.05))
+    (fp_line (start 0 0) (end 6.025 0) (layer "Edge.Cuts") (width 0.05))
+    (fp_line (start 9.925 0) (end 9.925 -3.5) (layer "Edge.Cuts") (width 0.05))
+    (fp_line (start -9.925 -3.5) (end -9.925 0) (layer "Edge.Cuts") (width 0.05))
+    (fp_line (start 10.425 -4) (end 11 -4) (layer "Edge.Cuts") (width 0.05))
+    (fp_line (start 7.225 -2.9) (end 7.225 0) (layer "Edge.Cuts") (width 0.05))
+    (fp_line (start -9.925 0) (end 0 0) (layer "Edge.Cuts") (width 0.05))
     (fp_line (start -11 -4) (end -10.425 -4) (layer "Edge.Cuts") (width 0.05))
-    (fp_line (start 3.225 -2.9) (end 3.225 0) (layer "Edge.Cuts") (width 0.05))
-    (fp_line (start -9.925 -3.5) (end -9.925 0) (layer "Edge.Cuts") (width 0.05))
-    (fp_line (start 0 0) (end 2.025 0) (layer "Edge.Cuts") (width 0.05))
-    (fp_line (start 9.925 0) (end 9.925 -3.5) (layer "Edge.Cuts") (width 0.05))
-    (fp_line (start 2.025 0) (end 2.025 -2.9) (layer "Edge.Cuts") (width 0.05))
-    (fp_line (start 10.425 -4) (end 11 -4) (layer "Edge.Cuts") (width 0.05))
-    (fp_line (start -9.925 0) (end 0 0) (layer "Edge.Cuts") (width 0.05))
-    (fp_line (start 3.225 0) (end 9.925 0) (layer "Edge.Cuts") (width 0.05))
+    (fp_line (start 6.025 0) (end 6.025 -2.9) (layer "Edge.Cuts") (width 0.05))
+    (fp_arc (start 6.025 -2.9) (mid 6.625 -3.5) (end 7.225 -2.9) (layer "Edge.Cuts") (width 0.05))
     (fp_arc (start 9.925 -3.5) (mid 10.071447 -3.853553) (end 10.425 -4) (layer "Edge.Cuts") (width 0.05))
-    (fp_arc (start 2.025 -2.9) (mid 2.625 -3.5) (end 3.225 -2.9) (layer "Edge.Cuts") (width 0.05))
     (fp_arc (start -10.425 -4) (mid -10.071447 -3.853553) (end -9.925 -3.5) (layer "Edge.Cuts") (width 0.05))
     (pad "1" smd rect (at 9.25 -1.275) (size 0.35 1.45) (layers "F.Cu"))
     (pad "2" smd rect (at 9 -1.525) (size 0.35 1.95) (layers "B.Cu"))
     (pad "3" smd rect (at 8.75 -1.275) (size 0.35 1.45) (layers "F.Cu"))
+    (pad "3V3" smd rect (at 4.025 -1.275) (size 0.35 1.45) (layers "F.Cu"))
     (pad "4" smd rect (at 8.5 -1.525) (size 0.35 1.95) (layers "B.Cu"))
     (pad "5" smd rect (at 8.25 -1.275) (size 0.35 1.45) (layers "F.Cu"))
     (pad "6" smd rect (at 8 -1.525) (size 0.35 1.95) (layers "B.Cu"))
     (pad "7" smd rect (at 7.75 -1.275) (size 0.35 1.45) (layers "F.Cu"))
-    (pad "8" smd rect (at 7.5 -1.525) (size 0.35 1.95) (layers "B.Cu"))
-    (pad "9" smd rect (at 7.25 -1.275) (size 0.35 1.45) (layers "F.Cu"))
-    (pad "10" smd rect (at 7 -1.525) (size 0.35 1.95) (layers "B.Cu"))
-    (pad "11" smd rect (at 6.75 -1.275) (size 0.35 1.45) (layers "F.Cu"))
-    (pad "12" smd rect (at 6.5 -1.525) (size 0.35 1.95) (layers "B.Cu"))
-    (pad "13" smd rect (at 6.25 -1.275) (size 0.35 1.45) (layers "F.Cu"))
-    (pad "14" smd rect (at 6 -1.525) (size 0.35 1.95) (layers "B.Cu"))
-    (pad "15" smd rect (at 5.75 -1.275) (size 0.35 1.45) (layers "F.Cu"))
+    (pad "12V" smd rect (at 4.275 -1.525) (size 0.35 1.95) (layers "B.Cu"))
     (pad "16" smd rect (at 5.5 -1.525) (size 0.35 1.95) (layers "B.Cu"))
     (pad "17" smd rect (at 5.25 -1.275) (size 0.35 1.45) (layers "F.Cu"))
@@
     (pad "22" smd rect (at 4 -1.525) (size 0.35 1.95) (layers "B.Cu"))
     (pad "23" smd rect (at 3.75 -1.275) (size 0.35 1.45) (layers "F.Cu"))
+    (pad "24" smd rect (at 3.5 -1.525) (size 0.35 1.95) (layers "B.Cu"))
+    (pad "25" smd rect (at 3.25 -1.275) (size 0.35 1.45) (layers "F.Cu"))
+    (pad "26" smd rect (at 3 -1.525) (size 0.35 1.95) (layers "B.Cu"))
+    (pad "27" smd rect (at 2.75 -1.275) (size 0.35 1.45) (layers "F.Cu"))
+    (pad "28" smd rect (at 2.5 -1.525) (size 0.35 1.95) (layers "B.Cu"))
+    (pad "29" smd rect (at 2.25 -1.275) (size 0.35 1.45) (layers "F.Cu"))
+    (pad "30" smd rect (at 2 -1.525) (size 0.35 1.95) (layers "B.Cu"))
+    (pad "31" smd rect (at 1.75 -1.275) (size 0.35 1.45) (layers "F.Cu"))
     (pad "32" smd rect (at 1.5 -1.525) (size 0.35 1.95) (layers "B.Cu"))
     (pad "33" smd rect (at 1.25 -1.275) (size 0.35 1.45) (layers "F.Cu"))
@@
     (pad "75" smd rect (at -9.25 -1.275) (size 0.35 1.45) (layers "F.Cu"))
   )
+  (footprint "NGFF:NGFF_2250" (layer "F.Cu")
+    (at 115 90)
+    (attr through_hole)
+    (fp_text reference "STOPs.top" (at -8 -49) (layer "F.SilkS")
+      (effects (font (size 0.5 0.5) (thickness 0.125)))
+    )
+    (fp_text value "2250" (at -8 -47.5) (layer "F.SilkS")
+      (effects (font (size 1 1) (thickness 0.15)))
+    )
+    (fp_line (start -11 -20) (end 11 -20) (layer "B.SilkS") (width 0.12))
+    (fp_line (start -11 -40) (end 11 -40) (layer "B.SilkS") (width 0.12))
+    (fp_line (start 0 0) (end 0 -30) (layer "Eco1.User") (width 0.01))
+    (fp_line (start 11 -50) (end 11 -4) (layer "Edge.Cuts") (width 0.05))
+    (fp_line (start 11 -50) (end -11 -50) (layer "Edge.Cuts") (width 0.05))
+    (fp_line (start -11 -50) (end -11 -4) (layer "Edge.Cuts") (width 0.05))
+    (fp_circle (center 0 -30) (end 1.5 -30) (layer "Edge.Cuts") (width 0.12) (fill none))
+    (fp_line (start -11 -50) (end -11 -4) (layer "F.CrtYd") (width 0.05))
+    (fp_line (start 11 -50) (end -11 -50) (layer "F.CrtYd") (width 0.05))
+    (fp_line (start 11 -50) (end 11 -4) (layer "F.CrtYd") (width 0.05))
+  )
 )

Commit message: update
Parts:
- removed STOPs.top: 2250, NGFF:NGFF_2250
- added NGFF2250: REF**, ngff:NGFF_2250, F.Cu at (115.0, 90.0)
Changed lines of the file:
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@@
     (at 115 90)
     (attr through_hole)
-    (fp_text reference "REF**" (at 5.6 2.07) (layer "F.SilkS")
+    (fp_text reference "REF**" (at 4 1.5) (layer "F.SilkS")
       (effects (font (size 1 1) (thickness 0.15)))
     )
-    (fp_text value "STOP_A" (at -0.075 2.05) (layer "F.Fab")
+    (fp_text value "STOP_A" (at -3 1.5) (layer "F.Fab")
       (effects (font (size 1 1) (thickness 0.15)))
     )
@@
     (pad "75" smd rect (at -9.25 -1.275) (size 0.35 1.45) (layers "F.Cu"))
   )
-  (footprint "NGFF:NGFF_2250" (layer "F.Cu")
+  (footprint "ngff:NGFF_2250" (layer "F.Cu")
     (at 115 90)
     (attr through_hole)
-    (fp_text reference "STOPs.top" (at -8 -49) (layer "F.SilkS")
+    (fp_text reference "NGFF2250" (at -0.05 -25.92) (layer "F.Fab")
       (effects (font (size 0.5 0.5) (thickness 0.125)))
     )
-    (fp_text value "2250" (at -8 -47.5) (layer "F.SilkS")
+    (fp_text value "REF**" (at 0.34 -27.21) (layer "F.SilkS")
       (effects (font (size 1 1) (thickness 0.15)))
     )
-    (fp_line (start -11 -20) (end 11 -20) (layer "B.SilkS") (width 0.12))
-    (fp_line (start -11 -40) (end 11 -40) (layer "B.SilkS") (width 0.12))
+    (fp_line (start 11 -30) (end -11 -30) (layer "B.SilkS") (width 0.12))
+    (fp_line (start -11 -42) (end 11 -42) (layer "B.SilkS") (width 0.12))
+    (fp_line (start -11 -22) (end 11 -22) (layer "B.SilkS") (width 0.12))
     (fp_line (start 0 0) (end 0 -30) (layer "Eco1.User") (width 0.01))
-    (fp_line (start 11 -50) (end 11 -4) (layer "Edge.Cuts") (width 0.05))
     (fp_line (start 11 -50) (end -11 -50) (layer "Edge.Cuts") (width 0.05))
     (fp_line (start -11 -50) (end -11 -4) (layer "Edge.Cuts") (width 0.05))
+    (fp_line (start 11 -50) (end 11 -4) (layer "Edge.Cuts") (width 0.05))
     (fp_circle (center 0 -30) (end 1.5 -30) (layer "Edge.Cuts") (width 0.12) (fill none))
-    (fp_line (start -11 -50) (end -11 -4) (layer "F.CrtYd") (width 0.05))
     (fp_line (start 11 -50) (end -11 -50) (layer "F.CrtYd") (width 0.05))
     (fp_line (start 11 -50) (end 11 -4) (layer "F.CrtYd") (width 0.05))
+    (fp_line (start -11 -50) (end -11 -4) (layer "F.CrtYd") (width 0.05))
   )
 )

Commit message: update
Parts:
- moved NGFF2250 18.0 mm to (100.0, 100.0)
- moved REF** 18.0 mm to (100.0, 100.0)
Other:
- rule pad_to_mask_clearance: 0.051 -> 0.05
Changed lines of the file:
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@@
 (kicad_pcb (version 20211014) (generator pcbnew)
   (general
-    (thickness 1.6)
+    (thickness 0.8)
   )
   (paper "A4")
@@
   )
   (setup
-    (pad_to_mask_clearance 0.051)
+    (pad_to_mask_clearance 0.05)
     (solder_mask_min_width 0.25)
+    (aux_axis_origin 100 100)
+    (grid_origin 100 100)
     (pcbplotparams
       (layerselection 0x00010fc_ffffffff)
@@
   (net 0 "")
   (footprint "ngff:NGFF_A" (layer "F.Cu")
-    (at 115 90)
+    (at 100 100)
     (attr through_hole)
     (fp_text reference "REF**" (at 4 1.5) (layer "F.SilkS")
@@
   )
   (footprint "ngff:NGFF_2250" (layer "F.Cu")
-    (at 115 90)
+    (at 100 100)
     (attr through_hole)
     (fp_text reference "NGFF2250" (at -0.05 -25.92) (layer "F.Fab")
