File: kicad/ngff.kicad_pcb (KiCad board)
At the start: 2 copper layers, 123.6 x 125.8 mm, 18 parts

Commit message: 更新更多款式
Parts:
- removed the STOPs.top at (275.3, 144.2)
- added STOPs.top: NGFF-2230, NGFF:m2-2230, F.Cu at (149.0, 111.0)
- STOPs.top (x6): footprint m2ngff:m2-outer2230 -> m2ngff:m2-2230
- STOPs.top: footprint m2ngff:m2-outer2230 -> NGFF:NGFF_2230
- STOPs.top: value NGFF-BM2230 -> NGFF-2230; footprint m2ngff:m2-outer2230 -> m2ngff:m2-2230
- moved REF** 157.7 mm to (45.7, 166.1)
- moved STOPs.top 157.7 mm to (45.7, 166.1)
- moved REF** 130.6 mm to (149.0, 111.0)
- moved REF** 129.6 mm to (114.8, 65.0)
- moved REF** 129.6 mm to (79.6, 116.1)
- moved STOPs.top 129.6 mm to (79.6, 116.1)
- moved STOPs.top 129.6 mm to (114.8, 65.0)
- moved AE 129.6 mm to (47.6, 116.7)
- moved REF** 129.6 mm to (147.5, 65.4)
- moved REF** 129.6 mm to (47.5, 65.2)
- moved REF** 129.6 mm to (77.9, 64.9)
- moved REF** 129.6 mm to (112.8, 114.8)
- moved STOPs.top 129.6 mm to (77.9, 64.9)
- moved STOPs.top 129.6 mm to (112.8, 114.8)
- moved STOPs.top 129.6 mm to (47.5, 65.2)
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Other:
- board size 123.6 x 125.8 mm -> 123.8 x 127.2 mm
