File: kicad/A2230.kicad_pcb (KiCad board)
At the start: 2 copper layers, 22 x 26 mm, 2 parts

Commit message: update
Parts:
- removed the REF** at (130.0, 90.0)
- removed STOPs.top: 2230, NGFF:NGFF_2230
- added NGFF2230: REF**, ngff:NGFF_2230, F.Cu at (100.0, 100.0)
- added REF**: STOP_A, ngff:NGFF_A, F.Cu at (100.0, 100.0)
Other:
- outline, holes or cut-outs redrawn
Changed lines of the file:
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@@
   )
   (net 0 "")
-  (footprint "NGFF:NGFF_2230" (layer "F.Cu")
-    (at 130 90)
-    (attr through_hole)
-    (fp_text reference "STOPs.top" (at -7.5 -28.5) (layer "F.SilkS")
-      (effects (font (size 0.5 0.5) (thickness 0.125)))
-    )
-    (fp_text value "2230" (at -7.5 -27) (layer "F.SilkS")
-      (effects (font (size 1 1) (thickness 0.15)))
-    )
-    (fp_line (start 0 0) (end 0 -30) (layer "Eco1.User") (width 0.01))
-    (fp_line (start 11 -30) (end 11 -4) (layer "Edge.Cuts") (width 0.05))
-    (fp_line (start 11 -30) (end -11 -30) (layer "Edge.Cuts") (width 0.05))
-    (fp_line (start -11 -30) (end -11 -4) (layer "Edge.Cuts") (width 0.05))
-    (fp_line (start -11 -30) (end -11 -4) (layer "F.CrtYd") (width 0.05))
-    (fp_line (start 11 -30) (end -11 -30) (layer "F.CrtYd") (width 0.05))
-    (fp_line (start 11 -30) (end 11 -4) (layer "F.CrtYd") (width 0.05))
-    (pad "1" thru_hole circle (at 0 -30) (size 5.5 5.5) (drill 3.5) (layers *.Cu *.Mask))
-  )
-  (footprint "NGFF:NGFF_A" (layer "F.Cu")
-    (at 130 90)
+  (footprint "ngff:NGFF_A" (layer "F.Cu")
+    (at 100 100)
     (attr through_hole)
     (fp_text reference "REF**" (at 5.6 2.07) (layer "F.SilkS")
       (effects (font (size 1 1) (thickness 0.15)))
     )
-    (fp_text value "NGFF_A" (at 0 2) (layer "F.Fab")
+    (fp_text value "STOP_A" (at -0.075 2.05) (layer "F.Fab")
       (effects (font (size 1 1) (thickness 0.15)))
     )
-    (fp_text user "A" (at 6.61 -3.94) (layer "F.SilkS")
+    (fp_text user "A" (at 6.675 -4) (layer "B.SilkS")
       (effects (font (size 0.8 0.8) (thickness 0.15)))
     )
+    (fp_poly (pts
+        (xy 7.225 0)
+        (xy 9.925 0)
+        (xy 9.925 -2.5)
+        (xy 7.225 -2.5)
+      ) (layer "B.Mask") (width 0.1) (fill solid))
     (fp_poly (pts
         (xy -9.925 0)
@@
         (xy 6.025 -2.5)
         (xy -9.925 -2.5)
-      ) (layer "B.Mask") (width 0.1) (fill solid))
-    (fp_poly (pts
-        (xy 7.225 0)
-        (xy 9.925 0)
-        (xy 9.925 -2.5)
-        (xy 7.225 -2.5)
       ) (layer "B.Mask") (width 0.1) (fill solid))
     (fp_poly (pts
@@
         (xy 7.225 -2)
       ) (layer "F.Mask") (width 0.1) (fill solid))
-    (fp_line (start -11 -4) (end -10.425 -4) (layer "Edge.Cuts") (width 0.05))
+    (fp_line (start 7.225 0) (end 9.925 0) (layer "Edge.Cuts") (width 0.05))
+    (fp_line (start 6.025 0) (end 6.025 -2.9) (layer "Edge.Cuts") (width 0.05))
     (fp_line (start 9.925 0) (end 9.925 -3.5) (layer "Edge.Cuts") (width 0.05))
-    (fp_line (start 7.225 0) (end 9.925 0) (layer "Edge.Cuts") (width 0.05))
-    (fp_line (start 0 0) (end 6.025 0) (layer "Edge.Cuts") (width 0.05))
-    (fp_line (start 6.025 0) (end 6.025 -2.9) (layer "Edge.Cuts") (width 0.05))
+    (fp_line (start 7.225 -2.9) (end 7.225 0) (layer "Edge.Cuts") (width 0.05))
     (fp_line (start 10.425 -4) (end 11 -4) (layer "Edge.Cuts") (width 0.05))
-    (fp_line (start 7.225 -2.9) (end 7.225 0) (layer "Edge.Cuts") (width 0.05))
     (fp_line (start -9.925 -3.5) (end -9.925 0) (layer "Edge.Cuts") (width 0.05))
     (fp_line (start -9.925 0) (end 0 0) (layer "Edge.Cuts") (width 0.05))
+    (fp_line (start -11 -4) (end -10.425 -4) (layer "Edge.Cuts") (width 0.05))
+    (fp_line (start 0 0) (end 6.025 0) (layer "Edge.Cuts") (width 0.05))
     (fp_arc (start 6.025 -2.9) (mid 6.625 -3.5) (end 7.225 -2.9) (layer "Edge.Cuts") (width 0.05))
     (fp_arc (start -10.425 -4) (mid -10.071447 -3.853553) (end -9.925 -3.5) (layer "Edge.Cuts") (width 0.05))
@@
     (pad "2" smd rect (at 9 -1.525) (size 0.35 1.95) (layers "B.Cu"))
     (pad "3" smd rect (at 8.75 -1.275) (size 0.35 1.45) (layers "F.Cu"))
+    (pad "3V3" smd rect (at 4.025 -1.275) (size 0.35 1.45) (layers "F.Cu"))
     (pad "4" smd rect (at 8.5 -1.525) (size 0.35 1.95) (layers "B.Cu"))
     (pad "5" smd rect (at 8.25 -1.275) (size 0.35 1.45) (layers "F.Cu"))
     (pad "6" smd rect (at 8 -1.525) (size 0.35 1.95) (layers "B.Cu"))
     (pad "7" smd rect (at 7.75 -1.275) (size 0.35 1.45) (layers "F.Cu"))
+    (pad "12V" smd rect (at 4.275 -1.525) (size 0.35 1.95) (layers "B.Cu"))
     (pad "16" smd rect (at 5.5 -1.525) (size 0.35 1.95) (layers "B.Cu"))
     (pad "17" smd rect (at 5.25 -1.275) (size 0.35 1.45) (layers "F.Cu"))
@@
     (pad "75" smd rect (at -9.25 -1.275) (size 0.35 1.45) (layers "F.Cu"))
   )
+  (footprint "ngff:NGFF_2230" (layer "F.Cu")
+    (at 100 100)
+    (attr through_hole)
+    (fp_text reference "NGFF2230" (at -0.03 -27.93) (layer "F.Fab")
+      (effects (font (size 0.5 0.5) (thickness 0.125)))
+    )
+    (fp_text value "REF**" (at 0.19 -26.62) (layer "F.SilkS")
+      (effects (font (size 1 1) (thickness 0.15)))
+    )
+    (fp_line (start -11 -20) (end 11 -20) (layer "B.SilkS") (width 0.12))
+    (fp_line (start 0 0) (end 0 -30) (layer "Eco1.User") (width 0.01))
+    (fp_line (start -1.5 -30) (end -11 -30) (layer "Edge.Cuts") (width 0.05))
+    (fp_line (start 11 -30) (end 1.5 -30) (layer "Edge.Cuts") (width 0.05))
+    (fp_line (start -11 -30) (end -11 -4) (layer "Edge.Cuts") (width 0.05))
+    (fp_line (start 11 -30) (end 11 -4) (layer "Edge.Cuts") (width 0.05))
+    (fp_arc (start 1.5 -30) (mid 0 -28.5) (end -1.5 -30) (layer "Edge.Cuts") (width 0.05))
+    (fp_line (start 11 -30) (end 11 -4) (layer "F.CrtYd") (width 0.05))
+    (fp_line (start 11 -30) (end -11 -30) (layer "F.CrtYd") (width 0.05))
+    (fp_line (start -11 -30) (end -11 -4) (layer "F.CrtYd") (width 0.05))
+  )
 )
